Commit message: Moved most of the joint control stuff to separate repo joint-control-pkgs

File: jaco_arm/jaco_gazebo/urdf/gzplugin_joint_control.urdf.xacro (robot description, xacro)
@@ -5,11 +5,30 @@
  xmlns:interface="http://playerstage.sourceforge.net/gazebo/xmlschema/#interface"
  xmlns:xacro="http://ros.org/wiki/xacro">
-<!-- MACRO FOR THE ROBOT ARM ON THE TABLE-->
-<xacro:macro name="gzplugin_joint_control">
+<!-- macro to laod jaco control plugins -->
+<xacro:macro name="gzplugin_joint_control" params="robot_components_namespace trajectory_param_namespace">
 	<gazebo>
-		<plugin name="gzplugin_joint_control" filename="libjaco_gazebo_joint_control.so"/>
-		<plugin name="gzplugin_joint_state_client" filename="libjaco_gazebo_joint_state_client.so"/>
-		<plugin name="gzplugin_joint_state_publisher" filename="libjaco_gazebo_joint_state_publisher.so"/>
-        <plugin name="gzplugin_joint_trajectory_server" filename="libjaco_gazebo_joint_trajectory_server.so"/>
+        <plugin name="gzplugin_joint_control" filename="libgazebo_joint_control.so">
+            <robot_components_namespace>
+                ${robot_components_namespace}
+            </robot_components_namespace>
+        </plugin>
+		<plugin name="gzplugin_joint_state_client" filename="libgazebo_joint_state_client.so">
+            <robot_components_namespace>
+                ${robot_components_namespace}
+            </robot_components_namespace>
+        </plugin>
+		<plugin name="gzplugin_joint_state_publisher" filename="libgazebo_joint_state_publisher.so">
+            <robot_components_namespace>
+                ${robot_components_namespace}
+            </robot_components_namespace>
+        </plugin>
+        <plugin name="gzplugin_joint_trajectory_server" filename="libgazebo_joint_trajectory_server.so">
+            <robot_components_namespace>
+                ${robot_components_namespace}
+            </robot_components_namespace>
+            <trajectory_param_namespace>
+                ${trajectory_param_namespace}
+            </trajectory_param_namespace>
+        </plugin>
 	</gazebo>
 </xacro:macro>

File: jaco_tutorial/jaco_on_table/urdf/jaco_on_table_robot_gazebo_ctrl.urdf.xacro (robot description, xacro)
@@ -4,4 +4,6 @@
 -->
 <robot name="JacoOnTable" xmlns:xacro="http://ros.org/wiki/xacro">
+    <xacro:arg name="robot_components_namespace" default="jaco"/>
+    <xacro:arg name="trajectory_param_namespace" default="jaco"/>
     <xacro:arg name="use_ros_control" default="false"/>
     <xacro:arg name="add_transmission_pos" default="false"/>
@@ -14,5 +16,8 @@
     </link>
 -->
-    <xacro:include filename="$(find jaco_on_table)/urdf/jaco_on_table.urdf.xacro" />
+    <xacro:include filename="$(find jaco_on_table)/urdf/jaco_on_table.urdf.xacro">
+        <xacro:arg name="add_transmission_pos" default="$(arg add_transmission_pos)"/>
+        <xacro:arg name="add_transmission_vel" default="$(arg add_transmission_vel)"/>
+    </xacro:include>
     <xacro:jaco_on_table parent="world">
         <origin xyz="0 0 0" rpy="0 0 0" />
@@ -20,13 +25,11 @@
     <xacro:if value="$(arg use_ros_control)">
         <xacro:include filename="$(find jaco_gazebo)/urdf/gzplugin_ros_control.urdf.xacro"/>
-        <xacro:arg name="add_transmission_pos" default="$(arg add_transmission_pos)"/>
-        <xacro:arg name="add_transmission_vel" default="$(arg add_transmission_vel)"/>
+        <xacro:gzplugin_joint_control/>
     </xacro:if>
     <xacro:unless value="$(arg use_ros_control)">
         <xacro:include filename="$(find jaco_gazebo)/urdf/gzplugin_joint_control.urdf.xacro"/>
-        <xacro:arg name="add_transmission_pos" default="$(arg add_transmission_pos)"/>
-        <xacro:arg name="add_transmission_vel" default="$(arg add_transmission_vel)"/>
+        <xacro:gzplugin_joint_control robot_components_namespace="$(arg robot_components_namespace)"
+                                  trajectory_param_namespace="$(arg trajectory_param_namespace)"/>
     </xacro:unless>
-    <xacro:gzplugin_joint_control/>
     <xacro:if value="$(arg load_grasp_fix)">
         <xacro:include filename="$(find jaco_gazebo)/urdf/gzplugin_grasp_fix.urdf.xacro"/>
