Commit message: small tidy up

File: jaco_arm/jaco_description/urdf/jaco.urdf.xacro (robot description, xacro)
@@ -97,5 +97,5 @@
 			</geometry>
 			<material name="">
-				<color rgba="0.109803921568627 0.109803921568627 0.109803921568627 1" />
+				<color rgba="0.10 0.10 0.10 1" />
 			</material>
 		</visual>
@@ -249,5 +249,5 @@
 			</geometry>
 			<material name="">
-				<color rgba="0.109803921568627 0.109803921568627 0.109803921568627 1" />
+				<color rgba="0.10 0.10 0.10 1" />
 			</material>
 		</visual>
@@ -270,5 +270,4 @@
 			<xacro:cyl_inertia mass="${0.00872/mass_divider}" h="0.02" r="0.04"/>
 		</inertial>
-<!--
 		<visual>
 			<origin xyz="0 0 0" rpy="0 0 0" />
@@ -277,8 +276,7 @@
 			</geometry>
 			<material name="">
-				<color rgba="0.501960784313725 0.501960784313725 0.501960784313725 1" />
-			</material>
-		</visual>
--->
+				<color rgba="0.50 0.50 0.50 1" />
+			</material>
+		</visual>
 		<collision>
 			<origin xyz="0 0 0" rpy="0 0 0" />
@@ -306,5 +304,5 @@
 			</geometry>
 			<material name="">
-				<color rgba="0.109803921568627 0.109803921568627 0.109803921568627 1" />
+				<color rgba="0.10 0.10 0.10 1" />
 			</material>
 		</visual>
@@ -337,5 +335,5 @@
 			</geometry>
 			<material name="">
-				<color rgba="0.501960784313725 0.501960784313725 0.501960784313725 1" />
+				<color rgba="0.50 0.50 0.50 1" />
 			</material>
 		</visual>
@@ -365,5 +363,5 @@
 			</geometry>
 			<material name="">
-				<color rgba="0.109803921568627 0.109803921568627 0.109803921568627 1" />
+				<color rgba="0.10 0.10 0.10 1" />
 			</material>
 		</visual>
@@ -396,5 +394,5 @@
 			</geometry>
 			<material name="">
-				<color rgba="0.501960784313725 0.501960784313725 0.501960784313725 1" />
+				<color rgba="0.5 0.5 0.5 1" />
 			</material>
 		</visual>
@@ -409,8 +407,8 @@
 		<origin xyz="0.41 0 0" rpy="${M_PI} 0 -${M_PI}" />
 		<parent link="2_upperarm_limb" />
-		<child link="ring_3" />
-		<axis xyz="0 0 0" />
-	</joint>
-	<!-- ...........................				-->
+		<child link="ring_3"/>
+		<axis xyz="0 0 0"/>
+	</joint>
+	<!-- ........................... -->
 	<link name="3_forearm_limb">
 		<inertial>
@@ -424,5 +422,5 @@
 			</geometry>
 			<material name="">
-				<color rgba="0.109803921568627 0.109803921568627 0.109803921568627 1" />
+				<color rgba="0.1 0.1 0.1 1" />
 			</material>
 		</visual>
@@ -455,5 +453,5 @@
 			</geometry>
 			<material name="">
-				<color rgba="0.501960784313725 0.501960784313725 0.501960784313725 1" />
+				<color rgba="0.5 0.5 0.5 1" />
 			</material>
 		</visual>
@@ -483,5 +481,5 @@
 			</geometry>
 			<material name="">
-				<color rgba="0.109803921568627 0.109803921568627 0.109803921568627 1" />
+				<color rgba="0.1 0.1 0.1 1" />
 			</material>
 		</visual>
@@ -514,5 +512,5 @@
 			</geometry>
 			<material name="">
-				<color rgba="0.501960784313725 0.501960784313725 0.501960784313725 1" />
+				<color rgba="0.5 0.5 0.5 1" />
 			</material>
 		</visual>
@@ -542,5 +540,5 @@
 			</geometry>
 			<material name="">
-				<color rgba="0.109803921568627 0.109803921568627 0.109803921568627 1" />
+				<color rgba="0.1 0.1 0.1 1" />
 			</material>
 		</visual>
@@ -575,5 +573,5 @@
 			</geometry>
 			<material name="">
-				<color rgba="0.501960784313725 0.501960784313725 0.501960784313725 1" />
+				<color rgba="0.5 0.5 0.5 1" />
 			</material>
 		</visual>
@@ -604,5 +602,5 @@
 			</geometry>
 			<material name="">
-				<color rgba="0.109803921568627 0.109803921568627 0.109803921568627 1" />
+				<color rgba="0.1 0.1 0.1 1" />
 			</material>
 		</visual>
@@ -651,5 +649,5 @@
 			</geometry>
 			<material name="">
-				<color rgba="0.501960784313725 0.501960784313725 0.501960784313725 1" />
+				<color rgba="0.5 0.5 0.5 1" />
 			</material>
 		</visual>
@@ -681,5 +679,5 @@
 			</geometry>
 			<material name="">
-				<color rgba="0.501960784313725 0.501960784313725 0.501960784313725 1" />
+				<color rgba="0.50 0.50 0.50 1" />
 			</material>
 		</visual>
@@ -712,5 +710,5 @@
 			</geometry>
 			<material name="">
-				<color rgba="0.501960784313725 0.501960784313725 0.501960784313725 1" />
+				<color rgba="0.5 0.5 0.5 1" />
 			</material>
 		</visual>
@@ -740,5 +738,5 @@
 			</geometry>
 			<material name="">
-				<color rgba="0.501960784313725 0.501960784313725 0.501960784313725 1" />
+				<color rgba="0.50 0.50 0.50 1" />
 			</material>
 		</visual>
@@ -769,5 +767,5 @@
 			</geometry>
 			<material name="">
-				<color rgba="0.501960784313725 0.501960784313725 0.501960784313725 1" />
+				<color rgba="0.5 0.5 0.5 1" />
 			</material>
 		</visual>
@@ -799,5 +797,5 @@
 			</geometry>
 			<material name="">
-				<color rgba="0.501960784313725 0.501960784313725 0.501960784313725 1" />
+				<color rgba="0.5 0.5 0.5 1" />
 			</material>
 		</visual>
@@ -827,5 +825,5 @@
 			</geometry>
 			<material name="">
-				<color rgba="0.501960784313725 0.501960784313725 0.501960784313725 1" />
+				<color rgba="0.5 0.5 0.5 1" />
 			</material>
 		</visual>
@@ -856,5 +854,5 @@
 			</geometry>
 			<material name="">
-				<color rgba="0.501960784313725 0.501960784313725 0.501960784313725 1" />
+				<color rgba="0.5 0.5 0.5 1" />
 			</material>
 		</visual>
@@ -886,5 +884,5 @@
 			</geometry>
 			<material name="">
-				<color rgba="0.501960784313725 0.501960784313725 0.501960784313725 1" />
+				<color rgba="0.5 0.5 0.5 1" />
 			</material>
 		</visual>

Commit message: Added example launch files for two arms, but no controllers supported yet

File: jaco_arm/jaco_description/urdf/jaco.urdf.xacro (robot description, xacro)
@@ -404,5 +404,5 @@
 		</collision>
 	</link>
-	<joint name="ring_3_joint" type="fixed">
+    <joint name="${jaco_prefix}_ring_3_joint" type="fixed">
 		<origin xyz="0.41 0 0" rpy="${M_PI} 0 -${M_PI}" />
         <parent link="${jaco_prefix}_2_upperarm_limb" />
@@ -522,5 +522,5 @@
 		</collision>
 	</link>
-	<joint name="ring_5_joint" type="fixed">
+    <joint name="${jaco_prefix}_ring_5_joint" type="fixed">
 		<origin xyz="-0.06590490 -0.034307921 0" rpy="-1.57079632679506 0 -0.610865238196312" />
         <parent link="${jaco_prefix}_4_upperwrist_limb" />

File: jaco_tutorial/jaco_on_table/urdf/jaco_on_table_robot.urdf (robot description, URDF)
Before this commit: robot JacoOnTable, 31 links, 30 joints
Joints:
- removed joint ring_3_joint
- removed joint ring_5_joint
- added joint jaco_ring_3_joint: type fixed, parent jaco_2_upperarm_limb, child jaco_ring_3, origin xyz=0.41 0 0 rpy=3.14159265359 0 -3.14159265359, axis 0 0 0
- added joint jaco_ring_5_joint: type fixed, parent jaco_4_upperwrist_limb, child jaco_ring_5, origin xyz=-0.06590490 -0.034307921 0 rpy=-1.57079632679506 0 -0.610865238196312, axis -1 0 0

File: jaco_tutorial/jaco_on_table/urdf/jaco_on_table_two_arms.urdf.xacro (robot description, xacro)
@@ -26,37 +26,30 @@
 	</joint>
     <xacro:include filename="$(find jaco_on_table)/urdf/objects/arm_stand.xacro" />
-    <xacro:arm_stand_link link_name="arm_stand"/>
-	<joint name="j2b" type="fixed">
-		<origin xyz="0 -0.035 0" rpy="-1.57079632679 -3.14159265358979 0" /> <!-- set the arm "inside" the table for now because of the rim along the real table. creating a bit of a buffer zone so moveit trajectories are within safe distance of the table edges. -->
+    <xacro:arm_stand_link link_name="arm_stand_left"/>
+    <xacro:arm_stand_link link_name="arm_stand_right"/>
+	<joint name="j2b1" type="fixed">
+        <origin xyz="0 -0.035 0" rpy="-1.57079632679 -3.14159265358979 0" />
 		<parent link="tabletop_corner" />
-		<child link="arm_stand" />
+		<child link="arm_stand_left" />
+		<axis xyz="0 0 0" />
+	</joint>
+	<joint name="j2b2" type="fixed">
+        <origin xyz="0.5 -0.035 0" rpy="-1.57079632679 -3.14159265358979 0" />
+		<parent link="tabletop_corner" />
+		<child link="arm_stand_right" />
 		<axis xyz="0 0 0" />
 	</joint>
 	<!-- Add the JACO arm to the given parent link with the given transforms -->
-	<xacro:include filename="$(find jaco_description)/urdf/jaco.urdf.xacro"/>
-    <xacro:jaco_arm parent="arm_stand" mass_divider="2" finger_mass_divider="1">
+    <xacro:include filename="$(find jaco_description)/urdf/jaco.urdf.xacro"/>
+    <xacro:jaco_arm parent="arm_stand_left" mass_divider="2" finger_mass_divider="1" jaco_prefix="jaco1">
+		<origin xyz="-0.000482247085224208 0.08 -0.000503436190578577" rpy="1.57079632679 0 3.14159265359" />
+        <xacro:arg name="add_transmission_pos" default="$(arg add_transmission_pos)"/>
+        <xacro:arg name="add_transmission_vel" default="$(arg add_transmission_vel)"/>
+    </xacro:jaco_arm>
+    <xacro:jaco_arm parent="arm_stand_right" mass_divider="2" finger_mass_divider="1" jaco_prefix="jaco2">
 		<origin xyz="-0.000482247085224208 0.08 -0.000503436190578577" rpy="1.57079632679 0 3.14159265359" />
         <xacro:arg name="add_transmission_pos" default="$(arg add_transmission_pos)"/>
         <xacro:arg name="add_transmission_vel" default="$(arg add_transmission_vel)"/>
 	</xacro:jaco_arm>
-<!-- Optional: Add the Xtion to the table to observe the real arm -->
-    <xacro:if value="$(arg sensor_on_table)">
-        <joint name="toxtion_base" type="fixed">
-            <origin xyz="0 -0.89 -0.01" rpy="0 0 -1.57079632679" />
-            <parent link="tabletop_corner" />
-            <child link="xtion_base" />
-        </joint>
-        <link name="xtion_base">
-            <visual>
-                <origin xyz="0 0 0" rpy="0 0 0" />
-                <geometry>
-                    <box size="0.02 0.02 0.02"/>
-                </geometry>
-                <material name="orange"/>
-            </visual>
-        </link>
-        <xacro:include filename="$(find common_sensors)/urdf/sensors/xtion_xtended_stand.urdf.xacro" />
-        <xacro:xtion_stand parent="xtion_base"/>
-    </xacro:if>
 </xacro:macro>
 </root>

File: jaco_tutorial/jaco_on_table/urdf/objects/arm_stand.xacro (robot description, xacro)
@@ -1,28 +1,30 @@
 <?xml version="1.0" encoding="UTF-8"?>
 <root xmlns:xacro="http://ros.org/wiki/xacro">
-    <gazebo reference="arm_stand">
-        <material>Gazebo/FlatBlack</material>
-    </gazebo>
-    <link name="arm_stand">
-        <inertial>
-            <origin xyz="2.55087129061304E-06 0.0160653225793 0.0184477855302965" rpy="0 0 0" />
-            <mass value="0.355288327861601" />
-            <inertia ixx="0.000857343821996639" ixy="6.2983660131078E-08" ixz="-3.19177822902163E-08" iyy="0.0019174970781523" iyz="-8.19713905978223E-05" izz="0.00176131215859239" />
-        </inertial>
-        <visual>
-            <origin xyz="0 0 0" rpy="0 0 0" />
-            <geometry>
-                <mesh filename="package://jaco_on_table/meshes/objects/arm_stand.STL" />
-            </geometry>
-            <material name="">
-                <color rgba="0.192156862745098 0.203921568627451 0.203921568627451 1" />
-            </material>
-        </visual>
-        <collision>
-            <origin xyz="0 0 0" rpy="0 0 0" />
-            <geometry>
-                <mesh filename="package://jaco_on_table/meshes/objects/arm_stand.STL" />
-            </geometry>
-        </collision>
-    </link>
+    <xacro:macro name="arm_stand_link" params="link_name">
+        <gazebo reference="${link_name}">
+            <material>Gazebo/FlatBlack</material>
+        </gazebo>
+        <link name="${link_name}">
+            <inertial>
+                <origin xyz="2.55087129061304E-06 0.0160653225793 0.0184477855302965" rpy="0 0 0" />
+                <mass value="0.355288327861601" />
+                <inertia ixx="0.000857343821996639" ixy="6.2983660131078E-08" ixz="-3.19177822902163E-08" iyy="0.0019174970781523" iyz="-8.19713905978223E-05" izz="0.00176131215859239" />
+            </inertial>
+            <visual>
+                <origin xyz="0 0 0" rpy="0 0 0" />
+                <geometry>
+                    <mesh filename="package://jaco_on_table/meshes/objects/arm_stand.STL" />
+                </geometry>
+                <material name="">
+                    <color rgba="0.192156862745098 0.203921568627451 0.203921568627451 1" />
+                </material>
+            </visual>
+            <collision>
+                <origin xyz="0 0 0" rpy="0 0 0" />
+                <geometry>
+                    <mesh filename="package://jaco_on_table/meshes/objects/arm_stand.STL" />
+                </geometry>
+            </collision>
+        </link>
+    </xacro:macro>
 </root>
