Commit message: Updated xacro files which had errors with properties inside macros

File: jaco_tutorial/jaco_on_table/urdf/jaco_on_table.urdf.xacro (robot description, xacro)
@@ -5,10 +5,13 @@
  xmlns:interface="http://playerstage.sourceforge.net/gazebo/xmlschema/#interface"
  xmlns:xacro="http://ros.org/wiki/xacro">
+<xacro:include filename="$(find jaco_on_table)/urdf/objects/table_properties.xacro" />
+<xacro:include filename="$(find jaco_on_table)/urdf/objects/arm_stand.xacro" />
+<xacro:include filename="$(find jaco_description)/urdf/jaco.urdf.xacro"/>
 <!-- MACRO FOR THE ROBOT ARM ON THE TABLE-->
 <xacro:macro name="jaco_on_table" params="parent *origin">
-    <xacro:arg name="sensor_on_table" default="false"/>
-    <!-- see jaco.urdf.xacro parameters of same name -->
-    <xacro:arg name="add_transmission_pos" default="false"/>
-    <xacro:arg name="add_transmission_vel" default="false"/>
+  <xacro:arg name="sensor_on_table" default="false"/>
+  <!-- see jaco.urdf.xacro parameters of same name -->
+  <xacro:arg name="add_transmission_pos" default="false"/>
+  <xacro:arg name="add_transmission_vel" default="false"/>
 	<joint name="base_to_jaco_on_table" type="fixed">
 		<xacro:insert_block name="origin" />
@@ -25,6 +28,5 @@
 		<child link="table_base"/>
 	</joint>
-    <xacro:include filename="$(find jaco_on_table)/urdf/objects/arm_stand.xacro" />
-    <xacro:arm_stand_link link_name="arm_stand"/>
+  <xacro:arm_stand_link link_name="arm_stand"/>
 	<joint name="j2b" type="fixed">
 		<origin xyz="0 -0.035 0" rpy="-1.57079632679 -3.14159265358979 0" /> <!-- set the arm "inside" the table for now because of the rim along the real table. creating a bit of a buffer zone so moveit trajectories are within safe distance of the table edges. -->
@@ -34,29 +36,28 @@
 	</joint>
 	<!-- Add the JACO arm to the given parent link with the given transforms -->
-	<xacro:include filename="$(find jaco_description)/urdf/jaco.urdf.xacro"/>
-    <xacro:jaco_arm parent="arm_stand" mass_divider="2" finger_mass_divider="1">
-		<origin xyz="-0.000482247085224208 0.08 -0.000503436190578577" rpy="1.57079632679 0 3.14159265359" />
-        <xacro:arg name="add_transmission_pos" default="$(arg add_transmission_pos)"/>
-        <xacro:arg name="add_transmission_vel" default="$(arg add_transmission_vel)"/>
+  <xacro:jaco_arm parent="arm_stand" mass_divider="2" finger_mass_divider="1">
+    <origin xyz="-0.000482247085224208 0.08 -0.000503436190578577" rpy="1.57079632679 0 3.14159265359" />
+    <xacro:arg name="add_transmission_pos" default="$(arg add_transmission_pos)"/>
+    <xacro:arg name="add_transmission_vel" default="$(arg add_transmission_vel)"/>
 	</xacro:jaco_arm>
-<!-- Optional: Add the Xtion to the table to observe the real arm -->
-    <xacro:if value="$(arg sensor_on_table)">
-        <joint name="toxtion_base" type="fixed">
-            <origin xyz="0 -0.89 -0.01" rpy="0 0 -1.57079632679" />
-            <parent link="tabletop_corner" />
-            <child link="xtion_base" />
-        </joint>
-        <link name="xtion_base">
-            <visual>
-                <origin xyz="0 0 0" rpy="0 0 0" />
-                <geometry>
-                    <box size="0.02 0.02 0.02"/>
-                </geometry>
-                <material name="orange"/>
-            </visual>
-        </link>
-        <xacro:include filename="$(find common_sensors)/urdf/sensors/xtion_xtended_stand.urdf.xacro" />
-        <xacro:xtion_stand parent="xtion_base"/>
-    </xacro:if>
+  <!-- Optional: Add the Xtion to the table to observe the real arm -->
+  <xacro:if value="$(arg sensor_on_table)">
+      <joint name="toxtion_base" type="fixed">
+          <origin xyz="0 -0.89 -0.01" rpy="0 0 -1.57079632679" />
+          <parent link="tabletop_corner" />
+          <child link="xtion_base" />
+      </joint>
+      <link name="xtion_base">
+          <visual>
+              <origin xyz="0 0 0" rpy="0 0 0" />
+              <geometry>
+                  <box size="0.02 0.02 0.02"/>
+              </geometry>
+              <material name="orange"/>
+          </visual>
+      </link>
+      <xacro:include filename="$(find common_sensors)/urdf/sensors/xtion_xtended_stand.urdf.xacro" />
+      <xacro:xtion_stand parent="xtion_base"/>
+  </xacro:if>
 </xacro:macro>
 </root>

File: jaco_tutorial/jaco_on_table/urdf/jaco_on_table_robot.urdf.xacro (robot description, xacro)
@@ -8,6 +8,6 @@
 	<link name="world"/>
 	<xacro:include filename="$(find jaco_on_table)/urdf/jaco_on_table.urdf.xacro" />
-    <xacro:jaco_on_table parent="world">
-        <origin xyz="0 0 0" rpy="0 0 0" />
-    </xacro:jaco_on_table>
+  <xacro:jaco_on_table parent="world">
+      <origin xyz="0 0 0" rpy="0 0 0" />
+  </xacro:jaco_on_table>
 </robot>

File: jaco_tutorial/jaco_on_table/urdf/objects/arm_stand.xacro (robot description, xacro)
@@ -1,30 +1,30 @@
 <?xml version="1.0" encoding="UTF-8"?>
 <root xmlns:xacro="http://ros.org/wiki/xacro">
-    <xacro:macro name="arm_stand_link" params="link_name">
-        <gazebo reference="${link_name}">
-            <material>Gazebo/FlatBlack</material>
-        </gazebo>
-        <link name="${link_name}">
-            <inertial>
-                <origin xyz="2.55087129061304E-06 0.0160653225793 0.0184477855302965" rpy="0 0 0" />
-                <mass value="0.355288327861601" />
-                <inertia ixx="0.000857343821996639" ixy="6.2983660131078E-08" ixz="-3.19177822902163E-08" iyy="0.0019174970781523" iyz="-8.19713905978223E-05" izz="0.00176131215859239" />
-            </inertial>
-            <visual>
-                <origin xyz="0 0 0" rpy="0 0 0" />
-                <geometry>
-                    <mesh filename="package://jaco_on_table/meshes/objects/arm_stand.STL" />
-                </geometry>
-                <material name="">
-                    <color rgba="0.192156862745098 0.203921568627451 0.203921568627451 1" />
-                </material>
-            </visual>
-            <collision>
-                <origin xyz="0 0 0" rpy="0 0 0" />
-                <geometry>
-                    <mesh filename="package://jaco_on_table/meshes/objects/arm_stand.STL" />
-                </geometry>
-            </collision>
-        </link>
-    </xacro:macro>
+  <xacro:macro name="arm_stand_link" params="link_name">
+    <gazebo reference="${link_name}">
+      <material>Gazebo/FlatBlack</material>
+    </gazebo>
+    <link name="${link_name}">
+      <inertial>
+        <origin xyz="2.55087129061304E-06 0.0160653225793 0.0184477855302965" rpy="0 0 0" />
+        <mass value="0.355288327861601" />
+        <inertia ixx="0.000857343821996639" ixy="6.2983660131078E-08" ixz="-3.19177822902163E-08" iyy="0.0019174970781523" iyz="-8.19713905978223E-05" izz="0.00176131215859239" />
+      </inertial>
+      <visual>
+        <origin xyz="0 0 0" rpy="0 0 0" />
+        <geometry>
+          <mesh filename="package://jaco_on_table/meshes/objects/arm_stand.STL" />
+        </geometry>
+        <material name="">
+          <color rgba="0.192156862745098 0.203921568627451 0.203921568627451 1" />
+        </material>
+      </visual>
+      <collision>
+        <origin xyz="0 0 0" rpy="0 0 0" />
+        <geometry>
+          <mesh filename="package://jaco_on_table/meshes/objects/arm_stand.STL" />
+        </geometry>
+      </collision>
+    </link>
+  </xacro:macro>
 </root>

File: jaco_tutorial/jaco_on_table/urdf/objects/table.xacro (robot description, xacro)
@@ -1,11 +1,5 @@
 <?xml version="1.0" encoding="UTF-8"?>
 <root xmlns:xacro="http://ros.org/wiki/xacro">
-	<xacro:macro name="default_material">
-	  <mu1>0.9</mu1>
-	  <mu2>0.9</mu2>
-		  <kp>1000000.0</kp>
-		  <kd>1.0</kd>
-	  <dynamics damping="0.7" friction="100.0" />
-	</xacro:macro>
+	<xacro:include filename="$(find jaco_on_table)/urdf/objects/table_properties.xacro" />
 	<gazebo reference="table_base">
 		<material>Gazebo/FlatBlack</material>
@@ -14,6 +8,4 @@
 		<material>Gazebo/White</material>
 	</gazebo>
-	<xacro:property name="table_width" value="0.8" />
-	<xacro:property name="table_length" value="1.05" />
 	<link name="table_base">
 		<inertial>
@@ -38,9 +30,4 @@
 		</collision>
 	</link>
-  <xacro:property name="t_width" value="1.05"/>
-  <xacro:property name="t_height" value="0.8"/>
-  <xacro:property name="t_thickness" value="0.03"/>
-  <xacro:property name="rim_height" value="0.015"/>
-  <xacro:property name="rim_thickness" value="0.005"/>
 	<link name="table_top">
 		<inertial>
